File: PCB/Thinkpad-USB-keyboard-PCB.kicad_pcb (KiCad board)
At the start: 2 copper layers, 86 x 33 mm, 55 parts, among them J1 TYPE-C-31-M12_13, J2 USB_A, J3 USB_A, J4 TYPE-C-31-M12_13, J6 TYPE-C-31-M12_13, U1 USBLC6-2SC6, U2 AP2112K-3.3, U3 USB2514B_Bi, U4 USBLC6-2SC6, U5 USBLC6-2SC6, U6 USBLC6-2SC6, U7 USBLC6-2SC6, Y1 Crystal_GND24

Commit message: More work
Parts:
- removed D2: 1N5819, Diode_SMD:D_SOD-123
- removed J6: TYPE-C-31-M12_13, AcheronConnectors:TYPE-C-31-M-12
- added C26: 100nF, Capacitor_SMD:C_0402_1005Metric, F.Cu at (87.6, 7.13)
- added J7: USB_C_Receptacle_USB2.0, Connector_USB:USB_C_Receptacle_HRO_TYPE-C-31-M-12, F.Cu at (85.4, -9.73)
- added R12: 100k, Resistor_SMD:R_0805_2012Metric_Pad1.20x1.40mm_HandSolder, F.Cu at (88.5, 4.67)
- added SW1: SW_Push, Button_Switch_THT:SW_PUSH_6mm_H5mm, F.Cu at (71.0, -13.5)
- added SW2: SW_Push, Button_Switch_THT:SW_PUSH_6mm_H5mm, F.Cu at (71.0, -4.95)
- added SW3: SW_Push, Connector_PinSocket_2.54mm:PinSocket_1x02_P2.54mm_Vertical, F.Cu at (71.3, 3.90)
- added U8: TLV1117-33, Package_TO_SOT_SMD:SOT-223-3_TabPin2, F.Cu at (84.5, -0.93)
- added Y2: Crystal_GND24, Crystal:Crystal_SMD_3225-4Pin_3.2x2.5mm_HandSoldering, F.Cu at (82.8, 6.02)
- J1: value TYPE-C-31-M12_13 -> USB_C_Receptacle_USB2.0; footprint AcheronConnectors:TYPE-C-31-M-12 -> Connector_USB:USB_C_Receptacle_HRO_TYPE-C-31-M-12
- R3: value 100k -> 27
- U2: value AP2112K-3.3 -> RP2040; footprint Package_TO_SOT_SMD:SOT-23-5 -> Package_DFN_QFN:QFN-56-1EP_7x7mm_P0.4mm_EP3.2x3.2mm
- U6: value USBLC6-2SC6 -> W25Q128JVS; footprint Package_TO_SOT_SMD:SOT-23-6 -> Package_SO:SOIC-8_5.23x5.23mm_P1.27mm
- moved U2 79.6 mm to (70.6, 19.4)
Connections:
- J1 pad A1: GNDPWR -> GND
- J1 pad B1: GNDPWR -> GND
- R1 pad 2: GNDPWR -> GND
- R2 pad 2: GNDPWR -> GND
- R3 pad 1: VCC -> D3+
- R3 pad 2: GND -> Net-(U2-USB_DP)
- U2 pad 1: VCC -> +3V3
- U2 pad 2: GND -> unconnected-(U2-GPIO0-Pad2)
- U2 pad 3: VCC -> unconnected-(U2-GPIO1-Pad3)
- U2 pad 5: +3V3 -> unconnected-(U2-GPIO3-Pad5)
- U3 pad 6: D3P- -> D3-
- U3 pad 7: D3P+ -> D3+
- U6 pad 1: D3P+ -> CS
- U6 pad 2: GND -> SD1
- U6 pad 3: D3P- -> SD2
- U6 pad 4: D3- -> GND
- U6 pad 5: VCC -> SD0
- U6 pad 6: D3+ -> QSPI_CLK

Commit message: More work
Parts:
- removed L3: 60R@100MHz, Inductor_SMD:L_1206_3216Metric
- removed R4: 1M, Resistor_SMD:R_0805_2012Metric_Pad1.15x1.40mm_HandSolder
- removed SW2: SW_Push, Button_Switch_THT:SW_PUSH_6mm_H5mm
- removed U7: USBLC6-2SC6, Package_TO_SOT_SMD:SOT-23-6
- added C27: 100nF, Capacitor_SMD:C_0402_1005Metric, F.Cu at (36.8, -41.2)
- added C28: 100nF, Capacitor_SMD:C_0402_1005Metric, F.Cu at (36.8, -39.2)
- added J6: Conn_02x20_Odd_Even_MountingPin, A-Thinkpad-USB-keyboard-footprints:Molex Slimstack 54363-0489, F.Cu at (34.6, 50.0)
- added U10: SRV05-4, Package_TO_SOT_SMD:SOT-23-6, F.Cu at (0.50, 8.80)
- C21: value 10u -> 1uF; footprint Capacitor_SMD:C_0805_2012Metric_Pad1.15x1.40mm_HandSolder -> Capacitor_SMD:C_0402_1005Metric
- J4: value TYPE-C-31-M12_13 -> SWD; footprint AcheronConnectors:TYPE-C-31-M-12 -> Connector_PinSocket_2.54mm:PinSocket_1x05_P2.54mm_Vertical
- U1, U4, U5: value USBLC6-2SC6 -> SRV05-4
- moved H6 75.6 mm to (93.3, -25.9)
- moved H3 66.0 mm to (84.3, -16.8)
- moved C26 62.4 mm to (87.1, -55.3)
- moved J4 62.4 mm to (48.5, -58.3)
- moved SW1 62.4 mm to (70.5, -75.9)
- moved Y2 62.4 mm to (82.3, -56.4)
- moved R12 62.4 mm to (88.0, -57.7)
- moved SW3 62.4 mm to (70.8, -58.5)
- moved U8 62.4 mm to (84.0, -63.3)
- moved H7 54.4 mm to (-80.0, -8.00)
- moved U5 45.8 mm to (27.9, 14.9), turned to 90 degrees
- moved C21 42.8 mm to (72.8, 22.0)
- moved H2 38.1 mm to (-71.0, 17.0)
- moved U4 37.4 mm to (7.70, 44.2)
- moved U2 37.3 mm to (34.6, 29.4), turned to 45 degrees
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Connections:
- C18 pad 1: VCC -> +5V
- C19 pad 1: VCC -> +5V
- C20 pad 1: VCC -> +5V
- C21 pad 1: VCC -> +1V1
- C5 pad 1: VCC -> +5V
- D1 pad 2: VCC -> +5V
- F1 pad 2: VCC -> +5V
- J2 pad 1: VCC -> +5V
- J3 pad 1: VCC -> +5V
- J7 pad A4: VBUS -> +5V
- J7 pad A6: D2+ -> D3+
- J7 pad A7: D2- -> D3-
- J7 pad A9: VBUS -> +5V
- J7 pad B4: VBUS -> +5V
- J7 pad B6: D2+ -> D3+
- J7 pad B7: D2- -> D3-
- J7 pad B9: VBUS -> +5V
- R3 pad 1: D3+ -> D2+
- SW1 pad 1: unconnected-(SW1-Pad1) -> GND
- SW1 pad 2: unconnected-(SW1-Pad2) -> +3V3
- U1 pad 1: DUP- -> D1+
- U1 pad 2: GNDPWR -> GND
- U1 pad 3: DUP+ -> D1-
- U1 pad 4: DUPP+ -> unconnected-(U1-IO3-Pad4)
- U1 pad 5: VBUS -> +5V
- U1 pad 6: DUPP- -> unconnected-(U1-IO4-Pad6)
- U2 pad 11: unconnected-(U2-GPIO8-Pad11) -> SENSE7
- U2 pad 12: PS2-DATA -> LED-CAPS-LOCK
- U2 pad 13: unconnected-(U2-GPIO10-Pad13) -> TP4-DATA
- U2 pad 14: PS2-CLK -> TP4-CLK
- U2 pad 15: unconnected-(U2-GPIO12-Pad15) -> LED-MIC-MUTE
- U2 pad 16: unconnected-(U2-GPIO13-Pad16) -> DRV13
- U2 pad 17: unconnected-(U2-GPIO14-Pad17) -> DRV15
- U2 pad 18: unconnected-(U2-GPIO15-Pad18) -> DRV12
- U2 pad 2: unconnected-(U2-GPIO0-Pad2) -> DRV4
- U2 pad 24: unconnected-(U2-SWCLK-Pad24) -> SWCLK
- U2 pad 25: unconnected-(U2-SWD-Pad25) -> SWD
- U2 pad 27: unconnected-(U2-GPIO16-Pad27) -> DRV14
- U2 pad 28: unconnected-(U2-GPIO17-Pad28) -> DRV11
- U2 pad 29: unconnected-(U2-GPIO18-Pad29) -> SENSE1
- U2 pad 3: unconnected-(U2-GPIO1-Pad3) -> DRV5
- U2 pad 30: unconnected-(U2-GPIO19-Pad30) -> SENSE4
- U2 pad 31: unconnected-(U2-GPIO20-Pad31) -> SENSE2
- U2 pad 32: unconnected-(U2-GPIO21-Pad32) -> SENSE3
- U2 pad 34: unconnected-(U2-GPIO22-Pad34) -> SENSE0
- U2 pad 35: unconnected-(U2-GPIO23-Pad35) -> SENSE5
- U2 pad 36: unconnected-(U2-GPIO24-Pad36) -> HOTKEY
- U2 pad 37: unconnected-(U2-GPIO25-Pad37) -> DRV10
- U2 pad 38: unconnected-(U2-GPIO26_ADC0-Pad38) -> DRV9
- U2 pad 39: unconnected-(U2-GPIO27_ADC1-Pad39) -> DRV0
- U2 pad 4: unconnected-(U2-GPIO2-Pad4) -> DRV8
- U2 pad 40: unconnected-(U2-GPIO28_ADC2-Pad40) -> DRV1
- U2 pad 5: unconnected-(U2-GPIO3-Pad5) -> DRV6
- U2 pad 6: unconnected-(U2-GPIO4-Pad6) -> DRV3
- U2 pad 7: unconnected-(U2-GPIO5-Pad7) -> DRV7
- U2 pad 8: unconnected-(U2-GPIO6-Pad8) -> DRV2
- U2 pad 9: unconnected-(U2-GPIO7-Pad9) -> SENSE6
- U3 pad 1: D1P- -> D1-
- U3 pad 2: D1P+ -> D1+
- U3 pad 3: D2P- -> D2-
- U3 pad 30: DUPP- -> DUP-
- U3 pad 31: DUPP+ -> DUP+
- U3 pad 4: D2P+ -> D2+
- U3 pad 8: D4P- -> D4-
- U3 pad 9: D4P+ -> D4+
- U4 pad 1: D1P+ -> unconnected-(U4-IO1-Pad1)
- U4 pad 3: D1P- -> unconnected-(U4-IO2-Pad3)
- U4 pad 4: D1- -> D3-
- U4 pad 5: VCC -> +5V
- U4 pad 6: D1+ -> D3+
- U5 pad 1: D2P+ -> unconnected-(U5-IO1-Pad1)
- U5 pad 3: D2P- -> unconnected-(U5-IO2-Pad3)
- U5 pad 4: D2- -> D4-
- U5 pad 5: VCC -> +5V
- U5 pad 6: D2+ -> D4+
- Y2 pad 1: Net-(U2-XIN) -> Net-(C9-Pad2)
- Y2 pad 3: Net-(C9-Pad2) -> Net-(U2-XIN)
Routing:
- net VCC: track 173.6 -> 0.00 mm, vias 4 -> 0
- net D3-: track 15.5 -> 63.5 mm
- net +5V: track 0.00 -> 45.7 mm, vias 0 -> 3
- net D1-: track 13.1 -> 58.7 mm
- net D3+: track 15.5 -> 60.0 mm
- net D1+: track 14.3 -> 58.7 mm
- net D2P+: track 37.0 -> 0.00 mm
- net D1P-: track 36.9 -> 0.00 mm
- net D1P+: track 36.0 -> 0.00 mm
- net D2P-: track 36.0 -> 0.00 mm
- net DRV11: track 0.00 -> 24.9 mm
- net D4-: track 4.58 -> 29.3 mm
- net SENSE6: track 0.00 -> 24.0 mm
- net DRV14: track 0.00 -> 23.9 mm
- net GND: track 10.2 -> 32.9 mm, vias 31 -> 19
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- added copper zone on B.Cu, net +5V
- added copper zone on F.Cu, net +5V
- removed copper zone on B.Cu, net VCC
- removed copper zone on F.Cu, net VCC
Other:
- board size 86 x 33 mm -> 85 x 1 mm

Commit message: More work
Parts:
- removed H10, H9: MountingHole, MountingHole:MountingHole_3.2mm_M3_ISO7380
- removed H11, H12: MountingHole, MountingHole:MountingHole_2.2mm_M2_ISO7380
- added C14: 10uF, Capacitor_SMD:C_1206_3216Metric_Pad1.33x1.80mm_HandSolder, F.Cu at (108.5, 27.4)
- added C15: 10uF, Capacitor_SMD:C_1206_3216Metric_Pad1.33x1.80mm_HandSolder, F.Cu at (108.5, 30.7)
- added C16: 10uF, Capacitor_SMD:C_1206_3216Metric_Pad1.33x1.80mm_HandSolder, F.Cu at (108.5, 34.1)
- added C17: 10uF, Capacitor_SMD:C_1206_3216Metric_Pad1.33x1.80mm_HandSolder, F.Cu at (108.5, 37.4)
- added C22: 100nF, Capacitor_SMD:C_0402_1005Metric_Pad0.74x0.62mm_HandSolder, F.Cu at (36.0, 25.5)
- added C23: 100nF, Capacitor_SMD:C_0402_1005Metric_Pad0.74x0.62mm_HandSolder, F.Cu at (30.0, 37.1)
- added C24: 100nF, Capacitor_SMD:C_0402_1005Metric_Pad0.74x0.62mm_HandSolder, F.Cu at (40.6, 34.3)
- added C25: 10uF, Capacitor_SMD:C_1206_3216Metric_Pad1.33x1.80mm_HandSolder, F.Cu at (34.1, 21.6)
- added C29: 1uF, Capacitor_SMD:C_0603_1608Metric_Pad1.08x0.95mm_HandSolder, F.Cu at (33.3, 23.6)
- added C30: 100nF, Capacitor_SMD:C_0402_1005Metric_Pad0.74x0.62mm_HandSolder, F.Cu at (39.5, 28.7)
- added C31: 100nF, Capacitor_SMD:C_0402_1005Metric_Pad0.74x0.62mm_HandSolder, F.Cu at (28.4, 32.2)
- added D3: RB060M-60TR, Diode_SMD:D_SOD-123, F.Cu at (88.8, 14.0)
- added D4: RB060M-60TR, Diode_SMD:D_SOD-123, F.Cu at (88.8, 17.4)
- added Q1: BSS138, Package_TO_SOT_SMD:SOT-23, F.Cu at (31.1, 41.4)
- added Q2: BSS138, Package_TO_SOT_SMD:SOT-23, F.Cu at (27.6, 43.5)
- added Q3: BSS138, Package_TO_SOT_SMD:SOT-23, F.Cu at (76.8, 56.5)
- added R10: 100, Resistor_SMD:R_0805_2012Metric_Pad1.20x1.40mm_HandSolder, F.Cu at (98.4, 33.1)
- added R11: 10K, Resistor_SMD:R_0603_1608Metric_Pad0.98x0.95mm_HandSolder, F.Cu at (33.9, 44.0)
- added R13: 27, Capacitor_SMD:C_0402_1005Metric_Pad0.74x0.62mm_HandSolder, F.Cu at (31.6, 26.0)
- added R14: 1K, Resistor_SMD:R_0805_2012Metric_Pad1.20x1.40mm_HandSolder, F.Cu at (43.0, 36.4)
- added R15: 1k, Resistor_SMD:R_0805_2012Metric_Pad1.20x1.40mm_HandSolder, F.Cu at (98.4, 41.9)
- added R16: 1k, Resistor_SMD:R_0805_2012Metric_Pad1.20x1.40mm_HandSolder, F.Cu at (103.1, 27.2)
- added R17: 4.7K, Resistor_SMD:R_0805_2012Metric_Pad1.20x1.40mm_HandSolder, F.Cu at (103.1, 30.1)
- added R18: 4.7K, Resistor_SMD:R_0805_2012Metric_Pad1.20x1.40mm_HandSolder, F.Cu at (103.1, 33.1)
- added R19: 10k, Resistor_SMD:R_0805_2012Metric_Pad1.20x1.40mm_HandSolder, F.Cu at (73.0, 66.5)
- added R20: 10K, Resistor_SMD:R_0603_1608Metric_Pad0.98x0.95mm_HandSolder, F.Cu at (32.3, 38.6)
- added R21: 10K, Resistor_SMD:R_0603_1608Metric_Pad0.98x0.95mm_HandSolder, F.Cu at (34.8, 42.4)
- added R22: 10K, Resistor_SMD:R_0603_1608Metric_Pad0.98x0.95mm_HandSolder, F.Cu at (102.5, 66.3)
- added R23: 10K, Resistor_SMD:R_0603_1608Metric_Pad0.98x0.95mm_HandSolder, F.Cu at (102.5, 69.3)
- added R4: 10K, Resistor_SMD:R_0603_1608Metric_Pad0.98x0.95mm_HandSolder, F.Cu at (33.6, 37.7)
- added R8: 56k, Resistor_SMD:R_0805_2012Metric_Pad1.20x1.40mm_HandSolder, F.Cu at (98.4, 27.2)
- added R9: 56k, Resistor_SMD:R_0805_2012Metric_Pad1.20x1.40mm_HandSolder, F.Cu at (98.4, 30.1)
- C1, C18, C19, C2, C20: value 10u -> 10uF; footprint Capacitor_SMD:C_0805_2012Metric_Pad1.15x1.40mm_HandSolder -> Capacitor_SMD:C_1206_3216Metric_Pad1.33x1.80mm_HandSolder
- C10, C11, C12, C13, C3, C4, C6, C7, C8: footprint Capacitor_SMD:C_0603_1608Metric_Pad1.05x0.95mm_HandSolder -> Capacitor_SMD:C_0402_1005Metric_Pad0.74x0.62mm_HandSolder
- C21: footprint Capacitor_SMD:C_0402_1005Metric -> Capacitor_SMD:C_0603_1608Metric_Pad1.08x0.95mm_HandSolder
- C26, C27, C28: footprint Capacitor_SMD:C_0402_1005Metric -> Capacitor_SMD:C_0402_1005Metric_Pad0.74x0.62mm_HandSolder
- C5, C9: value 1u -> 22pF; footprint Capacitor_SMD:C_0805_2012Metric_Pad1.15x1.40mm_HandSolder -> Capacitor_SMD:C_0402_1005Metric_Pad0.74x0.62mm_HandSolder
- D1: footprint AcheronComponents:D_SOD-123_Bidirectional -> Diode_SMD:D_SOD-123
- H1, H2, H3: value MountingHole -> MountingHole_Pad; footprint MountingHole:MountingHole_3.2mm_M3_ISO7380 -> MountingHole:MountingHole_3.2mm_M3_ISO7380_Pad
- H5: footprint MountingHole:MountingHole_2.2mm_M2_ISO7380_Pad -> MountingHole:MountingHole_3.2mm_M3_ISO7380_Pad
- H6, H7, H8: value MountingHole -> MountingHole_Pad; footprint MountingHole:MountingHole_2.2mm_M2_ISO7380 -> MountingHole:MountingHole_3.2mm_M3_ISO7380_Pad
- R1, R2, R5, R6, R7: footprint Resistor_SMD:R_0805_2012Metric_Pad1.15x1.40mm_HandSolder -> Resistor_SMD:R_0805_2012Metric_Pad1.20x1.40mm_HandSolder
- R3: footprint Resistor_SMD:R_0805_2012Metric_Pad1.15x1.40mm_HandSolder -> Capacitor_SMD:C_0402_1005Metric_Pad0.74x0.62mm_HandSolder
- moved H7 159.3 mm to (65.0, 58.0)
- moved H6 157.5 mm to (-40.0, 58.0)
- moved U8 136.3 mm to (-16.6, 28.7)
- moved C26 106.6 mm to (19.9, 27.5), turned to -90 degrees
- moved Y2 103.6 mm to (40.0, 38.1), turned to 135 degrees
- moved J4 102.4 mm to (53.0, 44.0)
- moved C28 72.9 mm to (41.3, 33.6), turned to -45 degrees
- moved H3 71.8 mm to (15.0, 2.00)
- moved C27 69.1 mm to (28.8, 27.5), turned to 135 degrees
- moved H8 64.8 mm to (0.00, 58.0)
- moved H2 57.0 mm to (-16.0, 2.00)
- moved C5 56.9 mm to (37.9, 40.2), turned to 135 degrees
- moved C9 53.6 mm to (42.3, 40.5), turned to 45 degrees
- moved R3 47.1 mm to (30.9, 26.7), turned to -45 degrees
- moved C21 40.8 mm to (32.1, 24.7), turned to 135 degrees
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Connections:
- C5 pad 1: +5V -> GND
- C5 pad 2: GND -> Net-(U2-XIN)
- C9 pad 1: +3V3 -> GND
- C9 pad 2: GND -> Net-(C9-Pad2)
- J6 pad 25: unconnected-(J6-Pin_25-Pad25) -> KBDID0
- J6 pad 27: unconnected-(J6-Pin_27-Pad27) -> KBDID1
- J6 pad 29: unconnected-(J6-Pin_29-Pad29) -> KBDID2
- J6 pad 33: unconnected-(J6-Pin_33-Pad33) -> LED-VOL-MUTE
- J6 pad 37: TP4-DATA -> TP4-DATA-5V
- J6 pad 39: TP4-CLK -> TP4-CLK-5V
- J6 pad 40: TP4-RESET -> TP4-RESET-5V
- U2 pad 11: SENSE7 -> PWRSWITCH
- U2 pad 13: TP4-DATA -> TP4-DATA-3V3
- U2 pad 14: TP4-CLK -> TP4-CLK-3V3
- U2 pad 15: LED-MIC-MUTE -> DRV13
- U2 pad 16: DRV13 -> DRV15
- U2 pad 17: DRV15 -> DRV12
- U2 pad 18: DRV12 -> DRV14
- U2 pad 2: DRV4 -> SENSE5
- U2 pad 27: DRV14 -> DRV11
- U2 pad 28: DRV11 -> DRV0
- U2 pad 29: SENSE1 -> DRV9
- U2 pad 3: DRV5 -> SENSE0
- U2 pad 30: SENSE4 -> DRV1
- U2 pad 31: SENSE2 -> DRV10
- U2 pad 32: SENSE3 -> DRV2
- U2 pad 34: SENSE0 -> DRV7
- U2 pad 35: SENSE5 -> DRV3
- U2 pad 36: HOTKEY -> DRV6
- U2 pad 37: DRV10 -> DRV8
- U2 pad 38: DRV9 -> DRV5
- U2 pad 39: DRV0 -> DRV4
- U2 pad 4: DRV8 -> SENSE3
- U2 pad 40: DRV1 -> HOTKEY
- U2 pad 41: unconnected-(U2-GPIO29_ADC3-Pad41) -> TP4-RESET-3V3
- U2 pad 5: DRV6 -> SENSE2
- U2 pad 6: DRV3 -> SENSE4
- U2 pad 7: DRV7 -> SENSE1
- U2 pad 8: DRV2 -> SENSE6
- U2 pad 9: SENSE6 -> SENSE7
Routing:
- net HOTKEY: track 0.00 -> 57.5 mm
- net DRV4: track 0.00 -> 47.0 mm
- net DRV5: track 0.00 -> 45.4 mm
- net DRV6: track 0.00 -> 43.9 mm
- net DRV8: track 0.00 -> 43.9 mm
- net DRV3: track 0.00 -> 42.3 mm
- net +3V3: track 77.5 -> 116.8 mm, vias 7 -> 9
- net DRV7: track 0.00 -> 39.2 mm
- net DRV2: track 0.00 -> 36.7 mm
- net DRV10: track 0.00 -> 35.1 mm
- net DRV1: track 0.00 -> 33.6 mm
- net SENSE5: track 0.00 -> 32.5 mm
- net DRV9: track 0.00 -> 32.0 mm
- net SENSE0: track 0.00 -> 31.6 mm
- net DRV0: track 0.00 -> 30.6 mm
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
Commit message: More work
Parts:
- moved U4 60.6 mm to (56.4, 8.10), turned to 90 degrees
- moved C19 14.7 mm to (-42.1, 18.6)
- moved C25 1.94 mm to (34.8, 23.4)
- moved C13 1.35 mm to (11.2, 22.7), turned to -45 degrees
- moved C23 1.09 mm to (30.0, 38.1)
- moved C24 1.09 mm to (40.6, 35.4)
- moved C28 1.09 mm to (41.3, 34.7)
- moved C31 1.09 mm to (28.4, 33.2)
- moved C5 1.09 mm to (37.9, 41.3)
- moved C9 1.09 mm to (42.3, 41.6)
- moved Q1 1.09 mm to (31.1, 42.5)
- moved Q2 1.09 mm to (27.6, 44.6)
- moved R4 1.09 mm to (33.6, 38.8)
- moved C11 1.09 mm to (29.8, 28.2)
- moved C22 1.09 mm to (36.0, 26.6)
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Routing:
- net GND: track 52.7 -> 83.8 mm, vias 27 -> 25
- net D2+: track 2.09 -> 27.3 mm
- net D2-: track 2.20 -> 26.4 mm
- net D3+: track 60.0 -> 65.0 mm
- net D3-: track 63.5 -> 66.6 mm
- net DUP+: track 21.6 -> 23.0 mm
- net D4-: track 29.3 -> 28.4 mm
- net DUP-: track 23.9 -> 23.1 mm
Other:
- board size 85 x 1 mm -> 111 x 64 mm

Commit message: More layout work
Parts:
- removed R19: 10k, Resistor_SMD:R_0805_2012Metric_Pad1.20x1.40mm_HandSolder
- added C32: 10uF, Capacitor_SMD:C_1206_3216Metric_Pad1.33x1.80mm_HandSolder, F.Cu at (18.1, 30.0)
- SW3: footprint Connector_PinSocket_2.54mm:PinSocket_1x02_P2.54mm_Vertical -> Button_Switch_THT:SW_PUSH_6mm_H5mm; moved to B.Cu
- moved C17 132.6 mm to (-22.4, 16.4), turned to 180 degrees
- moved C15 116.8 mm to (-7.81, 19.9), turned to -90 degrees
- moved C16 115.9 mm to (-5.99, 16.1)
- moved C14 115.4 mm to (-6.03, 13.3)
- moved SW3 107.8 mm to (13.3, 32.7), turned to 180 degrees
- moved D4 98.6 mm to (-9.82, 14.6), turned to -90 degrees
- moved R15 80.5 mm to (18.2, 35.2)
- moved SW1 76.9 mm to (120.7, -17.5)
- moved R16 51.8 mm to (55.7, 48.0)
- moved R22 46.6 mm to (61.2, 44.7)
- moved R23 46.0 mm to (60.3, 51.1), turned to 180 degrees
- moved C19 30.8 mm to (-12.6, 9.57), turned to -90 degrees
- moved Q3 17.8 mm to (61.3, 47.9)
- moved U8 13.0 mm to (-15.5, 15.7), turned to 180 degrees
- moved C23 1.26 mm to (31.0, 37.3)
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Connections:
- J4 pad 1: ~{RESET} -> RESET
- SW1 pad 2: +3V3 -> unconnected-(SW1-Pad2)
Routing:
- net +3V3: track 116.6 -> 269.4 mm, vias 9 -> 15
- net TP4-RESET-5V: track 0.00 -> 45.2 mm, vias 0 -> 2
- net TP4-RESET-3V3: track 3.13 -> 43.8 mm
- net SWD: track 4.43 -> 18.3 mm, vias 0 -> 1
- net +1V1: track 10.0 -> 23.8 mm, vias 0 -> 2
- net SWCLK: track 7.62 -> 21.3 mm, vias 0 -> 1
- net /~{USB_BOOT}: track 0.00 -> 11.3 mm
- net GND: track 83.8 -> 94.7 mm, vias 25 -> 60
- net +5V: track 46.1 -> 56.3 mm
- net D2-: track 26.4 -> 33.9 mm
- net D2+: track 27.3 -> 31.0 mm, vias 0 -> 2
- net CS: track 15.0 -> 17.2 mm
- net Net-(U3-XTALIN/CLKIN): track 14.6 -> 16.3 mm
- net HOTKEY: track 57.5 -> 58.2 mm
- net DRV11: track 29.9 -> 30.5 mm
