File: PCB/Thinkpad-USB-keyboard-PCB.kicad_pcb (KiCad board)
At the start: 2 copper layers, 111 x 64 mm, 89 parts, among them J1 USB_C_Receptacle_USB2.0, J2 USB_A, J3 USB_A, J4 SWD, J6 Conn_02x20_Odd_Even_MountingP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, J7 USB_C_Receptacle_USB2.0, Q1 BSS138, Q2 BSS138, Q3 BSS138, SW1 SW_Push, SW3 SW_Push, U1 SRV05-4, U10 SRV05-4, U2 RP2040, U3 USB2514B_Bi, U4 SRV05-4, U5 SRV05-4, U6 W25Q128JVS, U8 TLV1117-33, Y1 Crystal_GND24, Y2 Crystal_GND24

Commit message: More layout work
Parts:
- moved R9 51.9 mm to (52.5, 5.96), turned to 180 degrees
- moved R8 44.2 mm to (59.7, 5.81)
Routing:
- net +5V: track 56.3 -> 79.6 mm, vias 3 -> 7
- net Net-(J7-CC1): track 0.00 -> 2.94 mm
- net Net-(J7-CC2): track 0.00 -> 2.79 mm
Changed lines of the file:
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@@
   )
   (footprint "Resistor_SMD:R_0805_2012Metric_Pad1.20x1.40mm_HandSolder" (layer "F.Cu")
-    (at 98.3925 30.11)
+    (at 52.5 5.96 180)
     (descr "Resistor SMD 0805 (2012 Metric), square (rectangular) end terminal, IPC_7351 nominal with elongated pad for handsoldering. (Body size source: IPC-SM-782 page 72, https://www.pcb-3d.com/wordpress/wp-content/uploads/ipc-sm-782a_amendment_1_and_2.pdf), generated with kicad-footprint-generator")
     (tags "resistor handsolder")
@@
     (fp_line (start 1 0.625) (end -1 0.625)
       (stroke (width 0.1) (type solid)) (layer "F.Fab"))
-    (pad "1" smd roundrect (at -1 0) (size 1.2 1.4) (layers "F.Cu" "F.Paste" "F.Mask") (roundrect_rratio 0.208333)
+    (pad "1" smd roundrect (at -1 0 180) (size 1.2 1.4) (layers "F.Cu" "F.Paste" "F.Mask") (roundrect_rratio 0.208333)
       (net 48 "Net-(J7-CC2)") (pintype "passive"))
-    (pad "2" smd roundrect (at 1 0) (size 1.2 1.4) (layers "F.Cu" "F.Paste" "F.Mask") (roundrect_rratio 0.208333)
+    (pad "2" smd roundrect (at 1 0 180) (size 1.2 1.4) (layers "F.Cu" "F.Paste" "F.Mask") (roundrect_rratio 0.208333)
       (net 51 "+5V") (pintype "passive"))
     (model "${KICAD6_3DMODEL_DIR}/Resistor_SMD.3dshapes/R_0805_2012Metric.wrl"
@@
   )
   (footprint "Resistor_SMD:R_0805_2012Metric_Pad1.20x1.40mm_HandSolder" (layer "F.Cu")
-    (at 98.3925 27.16)
+    (at 59.74 5.81)
     (descr "Resistor SMD 0805 (2012 Metric), square (rectangular) end terminal, IPC_7351 nominal with elongated pad for handsoldering. (Body size source: IPC-SM-782 page 72, https://www.pcb-3d.com/wordpress/wp-content/uploads/ipc-sm-782a_amendment_1_and_2.pdf), generated with kicad-footprint-generator")
     (tags "resistor handsolder")
@@
   (segment (start 22.9752 50.078411) (end 29.146789 56.25) (width 0.2) (layer "F.Cu") (net 45))
   (segment (start 30.793057 33.830528) (end 22.9752 41.648385) (width 0.2) (layer "F.Cu") (net 45))
+  (segment (start 57.25 4.32) (end 57.25 3.485) (width 0.3) (layer "F.Cu") (net 46))
+  (segment (start 58.74 5.81) (end 57.25 4.32) (width 0.3) (layer "F.Cu") (net 46))
+  (segment (start 54.25 3.485) (end 54.25 5.21) (width 0.3) (layer "F.Cu") (net 48))
+  (segment (start 54.25 5.21) (end 53.5 5.96) (width 0.3) (layer "F.Cu") (net 48))
   (segment (start 32.490113 29.252012) (end 31.497811 28.25971) (width 0.2) (layer "F.Cu") (net 50))
   (segment (start 31.497811 28.25971) (end 31.214969 28.25971) (width 0.2) (layer "F.Cu") (net 50))
@@
   (segment (start -27.9 12.3) (end -28 12.2) (width 0.3) (layer "F.Cu") (net 51))
   (segment (start -7.5 9.46) (end -7.5 8.25) (width 0.75) (layer "F.Cu") (net 51))
+  (segment (start 53.55 2.69) (end 54.07 2.17) (width 0.3) (layer "F.Cu") (net 51))
+  (segment (start 53.55 3.485) (end 53.55 2.69) (width 0.3) (layer "F.Cu") (net 51))
   (segment (start -24 10.8125) (end -21.1425 13.67) (width 0.5) (layer "F.Cu") (net 51))
+  (segment (start 53.55 4.17) (end 53.55 3.485) (width 0.3) (layer "F.Cu") (net 51))
   (segment (start 35.75 43.484843) (end 35.69 43.484843) (width 0.3) (layer "F.Cu") (net 51))
+  (segment (start 60.74 5.81) (end 59.66 4.73) (width 0.3) (layer "F.Cu") (net 51))
   (segment (start 34.7625 44.412343) (end 34.7625 45.084843) (width 0.3) (layer "F.Cu") (net 51))
   (segment (start -12.31 9.46) (end -16.9325 9.46) (width 0.75) (layer "F.Cu") (net 51))
   (segment (start -6.15 0.9) (end -6.15 0.23) (width 0.75) (layer "F.Cu") (net 51))
   (segment (start -9.82 12.9025) (end -11.8125 12.9025) (width 1) (layer "F.Cu") (net 51))
+  (segment (start 58.45 2.73) (end 58.45 3.485) (width 0.3) (layer "F.Cu") (net 51))
   (segment (start -11.8125 12.9025) (end -12.34 13.43) (width 1) (layer "F.Cu") (net 51))
+  (segment (start 59.66 4.73) (end 58.89 4.73) (width 0.3) (layer "F.Cu") (net 51))
   (segment (start -8 12.9025) (end -7.5925 13.31) (width 1) (layer "F.Cu") (net 51))
   (segment (start -24.5 9.36) (end -24.5 9.384765) (width 0.5) (layer "F.Cu") (net 51))
+  (segment (start 58.45 4.29) (end 58.45 3.485) (width 0.3) (layer "F.Cu") (net 51))
+  (segment (start 58.89 4.73) (end 58.45 4.29) (width 0.3) (layer "F.Cu") (net 51))
   (segment (start -6.15 6.9) (end -6.15 0.9) (width 0.75) (layer "F.Cu") (net 51))
   (segment (start -9.82 12.9025) (end -9.82 9.62) (width 1) (layer "F.Cu") (net 51))
   (segment (start -6 7.05) (end -6.15 6.9) (width 0.75) (layer "F.Cu") (net 51))
+  (segment (start 60.74 4.67) (end 60.74 5.81) (width 0.3) (layer "F.Cu") (net 51))
   (segment (start 34.7625 48.037343) (end 35.48 48.754843) (width 0.3) (layer "F.Cu") (net 51))
   (segment (start -27.9 13.4625) (end -27.9 12.3) (width 0.3) (layer "F.Cu") (net 51))
   (segment (start 35.69 43.484843) (end 34.7625 44.412343) (width 0.3) (layer "F.Cu") (net 51))
+  (segment (start 56.37 7.81) (end 56.4 7.84) (width 0.3) (layer "F.Cu") (net 51))
+  (segment (start 57.86 2.14) (end 58.45 2.73) (width 0.3) (layer "F.Cu") (net 51))
   (segment (start -9.82 9.62) (end -9.98 9.46) (width 1) (layer "F.Cu") (net 51))
+  (segment (start 56.37 6.96) (end 56.37 7.81) (width 0.3) (layer "F.Cu") (net 51))
   (segment (start -12.63 9.14) (end -12.31 9.46) (width 1) (layer "F.Cu") (net 51))
+  (segment (start 51.5 5.96) (end 51.76 5.96) (width 0.3) (layer "F.Cu") (net 51))
+  (segment (start 51.76 5.96) (end 53.55 4.17) (width 0.3) (layer "F.Cu") (net 51))
   (segment (start -24 9.884765) (end -24 10.8125) (width 0.5) (layer "F.Cu") (net 51))
   (segment (start 35.484843 48.75) (end 37.7 48.75) (width 0.3) (layer "F.Cu") (net 51))
@@
   (segment (start -16.9325 9.46) (end -21.1425 13.67) (width 0.75) (layer "F.Cu") (net 51))
   (segment (start -12.63 8.0075) (end -12.63 9.14) (width 1) (layer "F.Cu") (net 51))
+  (via (at 56.4 7.84) (size 0.6) (drill 0.3) (layers "F.Cu" "B.Cu") (net 51))
   (via (at -28 12.2) (size 0.6) (drill 0.3) (layers "F.Cu" "B.Cu") (net 51))
   (via (at -6.15 0.9) (size 0.8) (drill 0.4) (layers "F.Cu" "B.Cu") (net 51))
+  (via (at 57.86 2.14) (size 0.6) (drill 0.3) (layers "F.Cu" "B.Cu") (net 51))
+  (via (at 54.07 2.17) (size 0.6) (drill 0.3) (layers "F.Cu" "B.Cu") (net 51))
   (via (at -6.15 -0.25) (size 0.8) (drill 0.4) (layers "F.Cu" "B.Cu") (net 51))
+  (via (at 60.74 4.67) (size 0.6) (drill 0.3) (layers "F.Cu" "B.Cu") (net 51))
+  (segment (start 56.4 6.22) (end 57.95 4.67) (width 0.3) (layer "B.Cu") (net 51))
   (segment (start -24.5 10.7) (end -24.5 9.36) (width 0.3) (layer "B.Cu") (net 51))
+  (segment (start 59.2 4.68) (end 59.21 4.67) (width 0.3) (layer "B.Cu") (net 51))
+  (segment (start 54.77 1.47) (end 57.19 1.47) (width 0.3) (layer "B.Cu") (net 51))
+  (segment (start 59.19 4.67) (end 59.2 4.68) (width 0.3) (layer "B.Cu") (net 51))
   (segment (start -26 11.1) (end -24.9 11.1) (width 0.3) (layer "B.Cu") (net 51))
   (segment (start -24.9 11.1) (end -24.5 10.7) (width 0.3) (layer "B.Cu") (net 51))
+  (segment (start 57.95 4.67) (end 59.19 4.67) (width 0.3) (layer "B.Cu") (net 51))
+  (segment (start 57.19 1.47) (end 57.86 2.14) (width 0.3) (layer "B.Cu") (net 51))
+  (segment (start 54.07 2.17) (end 54.77 1.47) (width 0.3) (layer "B.Cu") (net 51))
   (segment (start -28 12.2) (end -27.1 12.2) (width 0.3) (layer "B.Cu") (net 51))
+  (segment (start 56.4 7.84) (end 56.4 6.22) (width 0.3) (layer "B.Cu") (net 51))
   (segment (start -27.1 12.2) (end -26 11.1) (width 0.3) (layer "B.Cu") (net 51))
+  (segment (start 59.21 4.67) (end 60.74 4.67) (width 0.3) (layer "B.Cu") (net 51))
   (segment (start 42.841937 28.460043) (end 48.42 34.038106) (width 0.2) (layer "F.Cu") (net 52))
   (segment (start 39.144843 56.25) (end 37.7 56.25) (width 0.2) (layer "F.Cu") (net 52))

Commit message: More layout work
Parts:
- removed L2: 60R@100MHz, Inductor_SMD:L_1206_3216Metric
- removed R17, R18: 4.7K, Resistor_SMD:R_0805_2012Metric_Pad1.20x1.40mm_HandSolder
- added C33: 10uF, Capacitor_SMD:C_1206_3216Metric_Pad1.33x1.80mm_HandSolder, F.Cu at (63.6, 12.0)
- moved R12 123.7 mm to (-15.4, 10.1), turned to 90 degrees
- moved D3 98.5 mm to (-9.10, 3.10), turned to -90 degrees
- moved R10 72.4 mm to (28.0, 49.9), turned to 135 degrees
- moved R16 5.16 mm to (56.0, 42.8), turned to 90 degrees
- moved L1 1.24 mm to (8.00, 4.00)
- moved C25 0.49 mm to (34.5, 23.0)
Connections:
- R10 pad 1: LED-CAPS-LOCK -> LED-POWER
Routing:
- net GNDPWR: track 5.27 -> 179.0 mm, vias 3 -> 10
- net +5V: track 79.6 -> 248.2 mm, vias 7 -> 13
- net RESET: track 1.26 -> 60.7 mm, vias 1 -> 8
- net LED-POWER: track 0.00 -> 3.94 mm
- net GND: track 94.7 -> 98.4 mm, vias 60 -> 126
- net +3V3: track 269.4 -> 271.5 mm, vias 15 -> 18
- net +1V1: track 23.8 -> 23.3 mm
Other:
- board text added: "+3.3V"
- board text added: "GND"
- board text added: "RESET"
- board text added: "SWCLK"
- board text added: "SWD"
- board text added: "Thinkpad T410/etc keyboard to USB adapter Pylon 1/13/2024"

Commit message: Fixed some errors
Routing:
- net +5V: vias 13 -> 12
Changed lines of the file:
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@@
     (property "ki_keywords" "connector")
     (attr smd)
-    (fp_text reference "J6" (at 0 -20.32 unlocked) (layer "F.SilkS")
+    (fp_text reference "J6" (at -9.9 3.2 unlocked) (layer "User.1")
         (effects (font (size 1 1) (thickness 0.1)))
     )
@@
   (segment (start 34 29.1) (end 34 30.038077) (width 0.3) (layer "B.Cu") (net 2))
   (segment (start -2.45 2.65) (end -1.8 2) (width 0.5) (layer "F.Cu") (net 3))
-  (segment (start -4.7 8.5) (end -4.125 7.925) (width 0.5) (layer "F.Cu") (net 3))
-  (segment (start -2.75 7.2) (end -2.675 7.2) (width 0.5) (layer "F.Cu") (net 3))
   (segment (start 0.5 9.9375) (end 0.5 9.4) (width 0.3) (layer "F.Cu") (net 3))
+  (segment (start -3.06242 6.55) (end -3.06242 6.86242) (width 0.5) (layer "F.Cu") (net 3))
+  (segment (start -3.06242 4.91242) (end -3.06242 6.55) (width 0.5) (layer "F.Cu") (net 3))
   (segment (start -2.45 3.3975) (end -2.45 4.3) (width 0.5) (layer "F.Cu") (net 3))
   (segment (start 1.8 2) (end 2.45 2.65) (width 0.5) (layer "F.Cu") (net 3))
   (segment (start 0.5 9.4) (end 1.1 8.8) (width 0.3) (layer "F.Cu") (net 3))
   (segment (start -2.45 3.3975) (end -2.45 2.65) (width 0.5) (layer "F.Cu") (net 3))
-  (segment (start -3.06242 4.91242) (end -3.06242 6.88758) (width 0.5) (layer "F.Cu") (net 3))
-  (segment (start -3.06242 6.88758) (end -2.75 7.2) (width 0.5) (layer "F.Cu") (net 3))
+  (segment (start -3.06242 6.86242) (end -4.375 8.175) (width 0.5) (layer "F.Cu") (net 3))
   (segment (start -2.45 4.3) (end -3.06242 4.91242) (width 0.5) (layer "F.Cu") (net 3))
+  (segment (start -4.7 8.5) (end -4.375 8.175) (width 0.5) (layer "F.Cu") (net 3))
   (segment (start -4.7 9.46) (end -4.7 8.5) (width 0.5) (layer "F.Cu") (net 3))
-  (segment (start -4.125 7.925) (end -3.4 7.2) (width 0.75) (layer "F.Cu") (net 3))
+  (segment (start -4.375 8.175) (end -4.125 7.925) (width 0.5) (layer "F.Cu") (net 3))
   (segment (start 2.45 2.65) (end 2.45 3.3975) (width 0.5) (layer "F.Cu") (net 3))
-  (segment (start -3.4 7.2) (end -2.75 7.2) (width 0.75) (layer "F.Cu") (net 3))
   (via (at 1.1 8.8) (size 0.6) (drill 0.3) (layers "F.Cu" "B.Cu") (net 3))
   (via (at 1.8 2) (size 0.8) (drill 0.4) (layers "F.Cu" "B.Cu") (net 3))
@@
   (via (at -28 12.2) (size 0.6) (drill 0.3) (layers "F.Cu" "B.Cu") (net 51))
   (via (at 49.2 52.4) (size 0.6) (drill 0.3) (layers "F.Cu" "B.Cu") (net 51))
-  (via (at 42.7 46) (size 0.6) (drill 0.3) (layers "F.Cu" "B.Cu") (net 51))
   (via (at -6.15 0.9) (size 0.8) (drill 0.4) (layers "F.Cu" "B.Cu") (net 51))
   (via (at 57.86 2.14) (size 0.6) (drill 0.3) (layers "F.Cu" "B.Cu") (net 51))
