File: PCB/Thinkpad-USB-keyboard-PCB.kicad_pcb (KiCad board)
At the start: 2 copper layers, 111 x 64 mm, 87 parts, among them J1 USB_C_Receptacle_USB2.0, J2 USB_A, J3 USB_A, J4 SWD, J6 Conn_02x20_Odd_Even_MountingP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, J7 USB_C_Receptacle_USB2.0, Q1 BSS138, Q2 BSS138, Q3 BSS138, SW1 SW_Push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

Commit message: Finalized initial version
Parts:
- added C34: 10uF, Capacitor_SMD:C_1206_3216Metric_Pad1.33x1.80mm_HandSolder, F.Cu at (43.1, 43.2)
- added H10: MountingHole, A-Thinkpad-USB-keyboard-footprints:JLCPCB-tooling-hole, F.Cu at (59.0, 58.0)
- added H11: MountingHole, A-Thinkpad-USB-keyboard-footprints:JLCPCB-tooling-hole, F.Cu at (-37.0, 16.0)
- added H12: MountingHole, A-Thinkpad-USB-keyboard-footprints:JLCPCB-tooling-hole, F.Cu at (-35.0, 54.0)
- added H9: MountingHole, A-Thinkpad-USB-keyboard-footprints:JLCPCB-tooling-hole, F.Cu at (39.0, 0.00)
- added R17: DNI, Capacitor_SMD:C_0805_2012Metric_Pad1.18x1.45mm_HandSolder, F.Cu at (19.1, 38.2)
- added R18: 100, Resistor_SMD:R_0805_2012Metric_Pad1.20x1.40mm_HandSolder, F.Cu at (19.4, 48.8)
- added R19: 1M, Resistor_SMD:R_0805_2012Metric_Pad1.20x1.40mm_HandSolder, F.Cu at (3.90, 18.0)
- SW1: moved to B.Cu
- moved SW1 70.7 mm to (59.0, 17.0), turned to -90 degrees
- moved R1 0.81 mm to (3.70, 5.75)
- moved SW3 0.28 mm to (13.0, 32.7)
- moved R21 0.14 mm to (35.0, 43.5)
- moved R2 0.09 mm to (-3.08, 5.75)
Connections:
- SW1 pad 2: unconnected-(SW1-Pad2) -> RESET
- U2 pad 12: LED-CAPS-LOCK -> Net-(U2-GPIO9)
Routing:
- net Net-(U2-GPIO9): track 0.00 -> 21.2 mm, vias 0 -> 2
- net RESET: track 60.7 -> 72.5 mm
- net LED-CAPS-LOCK: track 24.0 -> 30.6 mm, vias 0 -> 2
- net GND: track 98.4 -> 93.6 mm, vias 126 -> 164
- net +3V3: track 271.5 -> 274.8 mm
- net +5V: track 248.2 -> 250.5 mm, vias 12 -> 13
- net CS: track 17.2 -> 19.1 mm
- net DRV3: track 42.3 -> 40.7 mm
- net D4+: track 27.1 -> 27.7 mm
- net Net-(J1-CC1): track 2.51 -> 3.16 mm
- net GNDPWR: vias 10 -> 14
Other:
- board text added: "BOOT"
- board text added: "JLCJLCJLCJLC"
- board text added: "Thinkpad T410/etc keyboard to USB adapter Pylon 1/14/2024"
- board text removed: "Thinkpad T410/etc keyboard to USB adapter Pylon 1/13/2024"

Commit message: finalized files
Parts:
- F1: footprint Fuse:Fuse_1206_3216Metric -> Fuse:Fuse_1812_4532Metric_Pad1.30x3.40mm_HandSolder
- R15, R16: value 1k -> 1K
- Y1: value Crystal_GND24 -> 24MHz
- Y2: value Crystal_GND24 -> 12MHz
- moved F1 0.98 mm to (-5.35, 10.1)
- moved R8 0.27 mm to (60.0, 5.89)
Routing:
- net LED-CAPS-LOCK: track 30.6 -> 27.6 mm
- net GND: vias 164 -> 163
Other:
- board text added: "Thinkpad T410/etc keyboard to USB adapter Pylon 1/15/2024"
- board text removed: "Thinkpad T410/etc keyboard to USB adapter Pylon 1/14/2024"
