File: PCB/Thinkpad-USB-keyboard-PCB.kicad_sch (KiCad schematic)
At the start: 80 parts, among them J1 USB_C_Receptacle_USB2.0, J2 USB_A, J3 USB_A, J4 SWD, J6 Conn_02x20_Odd_Even_MountingP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, J7 USB_C_Receptacle_USB2.0, SW1 SW_Push, SW3 SW_Push, U1 SRV05-4, U10 SRV05-4, U2 RP2040, U3 USB2514B_Bi, U4 SRV05-4, U5 SRV05-4, U6 W25Q128JVS, U8 TLV1117-33, Y1 Crystal_GND24, Y2 Crystal_GND24

Commit message: More layout work
Parts:
- removed R19: 10k, Resistor_SMD:R_0805_2012Metric_Pad1.20x1.40mm_HandSolder, symbol Device:R_Small
- added C32: 10uF, Capacitor_SMD:C_1206_3216Metric_Pad1.33x1.80mm_HandSolder, symbol Device:C
- SW3: footprint Connector_PinSocket_2.54mm:PinSocket_1x02_P2.54mm_Vertical -> Button_Switch_THT:SW_PUSH_6mm_H5mm
Connections:
- net +3V3: now also C32.1; no longer SW1.2
- net GND: now also C32.2
Other:
- moved on the sheet: C26
Changed lines of the file:
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@@
   (junction (at 491.49 172.72) (diameter 0) (color 0 0 0 0)
   )
-  (junction (at 436.88 388.62) (diameter 0) (color 0 0 0 0)
-  )
   (junction (at 105.41 158.75) (diameter 1.016) (color 0 0 0 0)
   )
@@
     (stroke (width 0) (type solid))
   )
-  (wire (pts (xy 436.88 386.08) (xy 436.88 388.62))
-    (stroke (width 0) (type default))
-  )
   (wire (pts (xy 284.48 60.96) (xy 284.48 59.69))
     (stroke (width 0) (type default))
@@
     (stroke (width 0) (type default))
   )
-  (wire (pts (xy 436.88 388.62) (xy 440.69 388.62))
-    (stroke (width 0) (type default))
-  )
   (wire (pts (xy 339.09 365.76) (xy 339.09 363.22))
     (stroke (width 0) (type default))
@@
     (stroke (width 0) (type solid))
   )
-  (wire (pts (xy 398.78 388.62) (xy 436.88 388.62))
+  (wire (pts (xy 398.78 388.62) (xy 440.69 388.62))
     (stroke (width 0) (type default))
   )
@@
     )
   )
+  (symbol (lib_id "power:+3.3V") (at 378.46 189.23 0) (unit 1)
+    (in_bom yes) (on_board yes) (dnp no)
+    (property "Reference" "#PWR070" (at 378.46 193.04 0)
+      (effects (font (size 1.27 1.27)) hide)
+    )
+    (property "Value" "+3.3V" (at 379.73 183.515 0)
+      (effects (font (size 1.27 1.27)))
+    )
+    (property "Footprint" "" (at 378.46 189.23 0)
+      (effects (font (size 1.27 1.27)) hide)
+    )
+    (property "Datasheet" "" (at 378.46 189.23 0)
+      (effects (font (size 1.27 1.27)) hide)
+    )
+    (pin "1")
+    (instances
+      (project "Thinkpad-USB-keyboard-PCB"
+        (path "/49b03f2e-4a93-4c4e-8d95-13775b5bcebc"
+          (reference "#PWR070") (unit 1)
+        )
+      )
+    )
+  )
   (symbol (lib_id "power:+3.3V") (at 80.01 201.295 0) (unit 1)
     (in_bom yes) (on_board yes) (dnp no)
@@
     )
   )
-  (symbol (lib_id "power:+3.3V") (at 372.11 199.39 0) (unit 1)
+  (symbol (lib_id "power:+3.3V") (at 369.57 190.5 0) (unit 1)
     (in_bom yes) (on_board yes) (dnp no)
-    (property "Reference" "#PWR062" (at 372.11 203.2 0)
+    (property "Reference" "#PWR062" (at 369.57 194.31 0)
       (effects (font (size 1.27 1.27)) hide)
     )
-    (property "Value" "+3.3V" (at 373.38 193.675 0)
+    (property "Value" "+3.3V" (at 370.84 184.785 0)
       (effects (font (size 1.27 1.27)))
     )
-    (property "Footprint" "" (at 372.11 199.39 0)
+    (property "Footprint" "" (at 369.57 190.5 0)
       (effects (font (size 1.27 1.27)) hide)
     )
-    (property "Datasheet" "" (at 372.11 199.39 0)
+    (property "Datasheet" "" (at 369.57 190.5 0)
       (effects (font (size 1.27 1.27)) hide)
     )
@@
     )
   )
+  (symbol (lib_id "Device:C") (at 378.46 193.04 0) (unit 1)
+    (in_bom yes) (on_board yes) (dnp no)
+    (property "Reference" "C32" (at 382.27 191.77 0)
+      (effects (font (size 1.27 1.27)) (justify left))
+    )
+    (property "Value" "10uF" (at 382.27 194.31 0)
+      (effects (font (size 1.27 1.27)) (justify left))
+    )
+    (property "Footprint" "Capacitor_SMD:C_1206_3216Metric_Pad1.33x1.80mm_HandSolder" (at 379.4252 196.85 0)
+      (effects (font (size 1.27 1.27)) hide)
+    )
+    (property "Datasheet" "~" (at 378.46 193.04 0)
+      (effects (font (size 1.27 1.27)) hide)
+    )
+    (pin "1")
+    (pin "2")
+    (instances
+      (project "Thinkpad-USB-keyboard-PCB"
+        (path "/49b03f2e-4a93-4c4e-8d95-13775b5bcebc"
+          (reference "C32") (unit 1)
+        )
+      )
+    )
+  )
   (symbol (lib_id "Device:C") (at 130.937 330.2 0) (unit 1)
     (in_bom yes) (on_board yes) (dnp no)
@@
     )
   )
-  (symbol (lib_id "power:+3.3V") (at 436.88 381 0) (unit 1)
-    (in_bom yes) (on_board yes) (dnp no)
-    (property "Reference" "#PWR045" (at 436.88 384.81 0)
-      (effects (font (size 1.27 1.27)) hide)
-    )
-    (property "Value" "+3.3V" (at 438.15 375.285 0)
-      (effects (font (size 1.27 1.27)))
-    )
-    (property "Footprint" "" (at 436.88 381 0)
-      (effects (font (size 1.27 1.27)) hide)
-    )
-    (property "Datasheet" "" (at 436.88 381 0)
-      (effects (font (size 1.27 1.27)) hide)
-    )
-    (pin "1")
-    (instances
-      (project "Thinkpad-USB-keyboard-PCB"
-        (path "/49b03f2e-4a93-4c4e-8d95-13775b5bcebc"
-          (reference "#PWR045") (unit 1)
-        )
-      )
-    )
-  )
   (symbol (lib_id "Device:R_Small") (at 370.84 44.45 90) (unit 1)
     (in_bom yes) (on_board yes) (dnp no)
@@
     )
   )
-  (symbol (lib_id "power:+3.3V") (at 297.18 274.32 0) (unit 1)
+  (symbol (lib_id "power:+3.3V") (at 297.18 271.78 0) (unit 1)
     (in_bom yes) (on_board yes) (dnp no)
-    (property "Reference" "#PWR016" (at 297.18 278.13 0)
+    (property "Reference" "#PWR016" (at 297.18 275.59 0)
       (effects (font (size 1.27 1.27)) hide)
     )
-    (property "Value" "+3.3V" (at 298.45 268.605 0)
+    (property "Value" "+3.3V" (at 298.45 266.065 0)
       (effects (font (size 1.27 1.27)))
     )
-    (property "Footprint" "" (at 297.18 274.32 0)
+    (property "Footprint" "" (at 297.18 271.78 0)
       (effects (font (size 1.27 1.27)) hide)
     )
-    (property "Datasheet" "" (at 297.18 274.32 0)
+    (property "Datasheet" "" (at 297.18 271.78 0)
       (effects (font (size 1.27 1.27)) hide)
     )
@@
     )
   )
-  (symbol (lib_id "Device:C_Small") (at 372.11 201.93 0) (unit 1)
+  (symbol (lib_id "Device:C_Small") (at 369.57 193.04 0) (unit 1)
     (in_bom yes) (on_board yes) (dnp no)
-    (property "Reference" "C26" (at 373.38 200.6599 90)
+    (property "Reference" "C26" (at 370.84 191.7699 90)
       (effects (font (size 1.27 1.27)) (justify left))
     )
-    (property "Value" "100nF" (at 373.38 209.5499 90)
+    (property "Value" "100nF" (at 370.84 200.6599 90)
       (effects (font (size 1.27 1.27)) (justify left))
     )
-    (property "Footprint" "Capacitor_SMD:C_0402_1005Metric_Pad0.74x0.62mm_HandSolder" (at 372.11 201.93 0)
+    (property "Footprint" "Capacitor_SMD:C_0402_1005Metric_Pad0.74x0.62mm_HandSolder" (at 369.57 193.04 0)
       (effects (font (size 1.27 1.27)) hide)
     )
-    (property "Datasheet" "~" (at 372.11 201.93 0)
+    (property "Datasheet" "~" (at 369.57 193.04 0)
       (effects (font (size 1.27 1.27)) hide)
     )
-    (property "LCSC" "C1525" (at 372.11 201.93 0)
+    (property "LCSC" "C1525" (at 369.57 193.04 0)
       (effects (font (size 1.27 1.27)) hide)
     )
@@
     )
   )
-  (symbol (lib_id "Device:R_Small") (at 436.88 383.54 180) (unit 1)
-    (in_bom yes) (on_board yes) (dnp no)
-    (property "Reference" "R19" (at 434.34 383.54 90)
-      (effects (font (size 1.27 1.27)))
-    )
-    (property "Value" "10k" (at 439.42 383.54 90)
-      (effects (font (size 1.27 1.27)))
-    )
-    (property "Footprint" "Resistor_SMD:R_0805_2012Metric_Pad1.20x1.40mm_HandSolder" (at 436.88 383.54 0)
-      (effects (font (size 1.27 1.27)) hide)
-    )
-    (property "Datasheet" "~" (at 436.88 383.54 0)
-      (effects (font (size 1.27 1.27)) hide)
-    )
-    (property "LCSC" "C11702" (at 436.88 383.54 0)
-      (effects (font (size 1.27 1.27)) hide)
-    )
-    (pin "1")
-    (pin "2")
-    (instances
-      (project "Thinkpad-USB-keyboard-PCB"
-        (path "/49b03f2e-4a93-4c4e-8d95-13775b5bcebc"
-          (reference "R19") (unit 1)
-        )
-      )
-    )
-  )
   (symbol (lib_id "power:GND") (at 53.34 48.26 0) (unit 1)
     (in_bom yes) (on_board yes) (dnp no)
@@
     )
   )
-  (symbol (lib_id "power:GND") (at 372.11 204.47 0) (unit 1)
+  (symbol (lib_id "power:GND") (at 369.57 195.58 0) (unit 1)
     (in_bom yes) (on_board yes) (dnp no)
-    (property "Reference" "#PWR039" (at 372.11 210.82 0)
+    (property "Reference" "#PWR039" (at 369.57 201.93 0)
       (effects (font (size 1.27 1.27)) hide)
     )
-    (property "Value" "GND" (at 377.19 204.47 0)
+    (property "Value" "GND" (at 374.65 195.58 0)
       (effects (font (size 1.27 1.27)))
     )
-    (property "Footprint" "" (at 372.11 204.47 0)
+    (property "Footprint" "" (at 369.57 195.58 0)
       (effects (font (size 1.27 1.27)) hide)
     )
-    (property "Datasheet" "" (at 372.11 204.47 0)
+    (property "Datasheet" "" (at 369.57 195.58 0)
       (effects (font (size 1.27 1.27)) hide)
     )
@@
       (effects (font (size 1.27 1.27)))
     )
-    (property "Footprint" "Connector_PinSocket_2.54mm:PinSocket_1x02_P2.54mm_Vertical" (at 324.485 208.28 0)
+    (property "Footprint" "Button_Switch_THT:SW_PUSH_6mm_H5mm" (at 324.485 208.28 0)
       (effects (font (size 1.27 1.27)) hide)
     )
@@
         )
       )
+    )
+  )
+  (symbol (lib_id "power:GND") (at 378.46 196.85 0) (unit 1)
+    (in_bom yes) (on_board yes) (dnp no)
+    (property "Reference" "#PWR071" (at 378.46 203.2 0)
+      (effects (font (size 1.27 1.27)) hide)
+    )
+    (property "Value" "GND" (at 383.54 196.85 0)
+      (effects (font (size 1.27 1.27)))
+    )
+    (property "Footprint" "" (at 378.46 196.85 0)
+      (effects (font (size 1.27 1.27)) hide)
+    )
+    (property "Datasheet" "" (at 378.46 196.85 0)
+      (effects (font (size 1.27 1.27)) hide)
+    )
+    (pin "1")
+    (instances
+      (project "Thinkpad-USB-keyboard-PCB"
+        (path "/49b03f2e-4a93-4c4e-8d95-13775b5bcebc"
+          (reference "#PWR071") (unit 1)
+        )
+      )

Commit message: More layout work
Parts:
- removed L2: 60R@100MHz, Inductor_SMD:L_1206_3216Metric, symbol Unified-Daughterboard-rescue:L_Core_Ferrite-Device
- removed R17, R18: 4.7K, Resistor_SMD:R_0805_2012Metric_Pad1.20x1.40mm_HandSolder, symbol Device:R_Small
- added C33: 10uF, Capacitor_SMD:C_1206_3216Metric_Pad1.33x1.80mm_HandSolder, symbol Device:C
Connections:
- net ~{RESET} is gone; now on net RESET: J4.1 (Pin_1)
- net +5V: now also C33.1
- net GND: now also C33.2
- net LED-CAPS-LOCK: no longer R10.1
- net LED-POWER: now also R10.1

Commit message: Finalized initial version
Parts:
- added C34: 10uF, Capacitor_SMD:C_1206_3216Metric_Pad1.33x1.80mm_HandSolder, symbol Device:C
- added H10, H11, H12, H9: MountingHole, A-Thinkpad-USB-keyboard-footprints:JLCPCB-tooling-hole, symbol Mechanical:MountingHole
- added R17: DNI, Capacitor_SMD:C_0805_2012Metric_Pad1.18x1.45mm_HandSolder, symbol Device:R
- added R18: 100, Resistor_SMD:R_0805_2012Metric_Pad1.20x1.40mm_HandSolder, symbol Device:R_Small
- added R19: 1M, Resistor_SMD:R_0805_2012Metric_Pad1.20x1.40mm_HandSolder, symbol Device:R
Connections:
- net +3V3: now also R17.2
- net +5V: now also C34.1
- net CS: now also R17.1
- net GND: now also C34.2
- net LED-CAPS-LOCK: now also R18.1; no longer U2.12 (GPIO9)
- net RESET: now also SW1.2
- net at C3.2, U3.33 (XTALIN/CLKIN), Y1.1: now also R19.1
- net at C4.2, U3.32 (XTALOUT), Y1.3: now also R19.2
- new net: R18.2, U2.12 (GPIO9)
Other:
- note added: "JLCPCB tooling holes"
- note added: "RP2040"
- note added: "Thinkpad connector"
- moved on the sheet: C11, C14, C15, C16, C17, C18, C19, C20, C21, C22, C23, C24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

Commit message: finalized files
Parts:
- F1: value ASMD1206-150 -> 1812L075PR; footprint Fuse:Fuse_1206_3216Metric -> Fuse:Fuse_1812_4532Metric_Pad1.30x3.40mm_HandSolder
- R15, R16: value 1k -> 1K
- Y1: value Crystal_GND24 -> 24MHz
- Y2: value Crystal_GND24 -> 12MHz
Changed lines of the file:
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@@
       (effects (font (size 1.27 1.27)))
     )
-    (property "Value" "ASMD1206-150" (at 121.285 50.5714 90)
+    (property "Value" "1812L075PR" (at 121.285 50.5714 90)
       (effects (font (size 0.508 0.508)))
     )
-    (property "Footprint" "Fuse:Fuse_1206_3216Metric" (at 126.365 52.07 0)
+    (property "Footprint" "Fuse:Fuse_1812_4532Metric_Pad1.30x3.40mm_HandSolder" (at 126.365 52.07 0)
       (effects (font (size 1.27 1.27)) (justify left) hide)
     )
@@
       (effects (font (size 1.27 1.27)))
     )
-    (property "Value" "1k" (at 218.44 223.52 90)
+    (property "Value" "1K" (at 218.44 223.52 90)
       (effects (font (size 1.27 1.27)))
     )
@@
       (effects (font (size 1.27 1.27)) (justify left))
     )
-    (property "Value" "Crystal_GND24" (at 39.37 255.905 90)
+    (property "Value" "24MHz" (at 39.37 255.905 90)
       (effects (font (size 1.27 1.27)) (justify left))
     )
@@
       (effects (font (size 1.27 1.27)) (justify left))
     )
-    (property "Value" "Crystal_GND24" (at 297.18 266.7 90)
+    (property "Value" "12MHz" (at 297.18 266.7 90)
       (effects (font (size 1.27 1.27)) (justify left))
     )
@@
       (effects (font (size 1.27 1.27)))
     )
-    (property "Value" "1k" (at 302.26 213.36 90)
-      (effects (font (size 1.27 1.27)))
-    )
+    (property "Value" "1K" (at 302.26 213.36 90)
+      (effects (font (size 1.27 1.27)))
+    )
