File: Thinkpad keyboard connector breakout/Keyboard-connector-breakout/Keyboard-connector-breakout.kicad_pcb (KiCad board)
At the start: 2 copper layers, 26 x 54 mm, 8 parts, among them J1 Conn_02x20_Odd_Even_MountingP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, J2 Conn_01x20_Socket, J3 Conn_01x20_Socket, J4 Conn_01x01_Socket

Commit message: More work
Other:
- board text added: "GND"
Changed lines of the file:
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@@
     (property "ki_keywords" "connector")
     (attr through_hole)
-    (fp_text reference "J4" (at 0 -2.33 90) (layer "F.SilkS")
+    (fp_text reference "J4" (at 0 -2.33 90) (layer "Dwgs.User")
         (effects (font (size 1 1) (thickness 0.15)))
     )
@@
     (property "ki_keywords" "connector")
     (attr through_hole)
-    (fp_text reference "J3" (at 0 -2.77) (layer "F.SilkS")
+    (fp_text reference "J3" (at 0 -2.77) (layer "Dwgs.User")
         (effects (font (size 1 1) (thickness 0.15)))
     )
@@
     (property "ki_keywords" "connector")
     (attr through_hole)
-    (fp_text reference "J2" (at 0 -2.77) (layer "F.SilkS")
+    (fp_text reference "J2" (at 0 -1.87) (layer "Dwgs.User")
         (effects (font (size 1 1) (thickness 0.15)))
     )
@@
     (effects (font (size 1.5 1.5) (thickness 0.3) bold) (justify left bottom))
   )
+  (gr_text "GND" (at 0 -23) (layer "F.SilkS")
+    (effects (font (size 1 1) (thickness 0.15)) (justify left bottom))
+  )
   (segment (start -4.325 -18.295) (end -4.325 -5.075001) (width 0.25) (layer "F.Cu") (net 1))
